File: Schaltplan/Schaltplan.kicad_sch (KiCad schematic)
At the start: 9 parts, among them J2 Buck Converter, M2 Stepper_Motor_bipolar, M3 Stepper_Motor_bipolar

Commit message: New file names
Parts:
- added R1, R2: R, symbol Device:R
- renumbered U3 to U3RIGHT, U4 to U4LEFT
Connections:
- net +11.1V: now also R1.1
- net +5V: no longer U3RIGHT.2 (GND), U3RIGHT.3 (A2), U4LEFT.2 (GND), U4LEFT.3 (A2)
- net GND: now also R2.2; no longer U3RIGHT.1 (VM), U4LEFT.1 (VM)
- net at U3RIGHT.4 (A1): now also M2.1
- net at U3RIGHT.5 (B1): now also M2.4
- net at U3RIGHT.6 (B2): now also M2.3
- net GPIO 16: now reaches U3RIGHT.7 (VCC_IO)
- net GPIO 16: no longer U1.12 (GPIO34)
- net GPIO 17: now reaches U3RIGHT.8 (GND)
- net GPIO 17: no longer U1.13 (GPIO39)
- net at U4LEFT.4 (A1): now also M3.1
- net at U4LEFT.5 (B1): now also M3.4
- net at U4LEFT.6 (B2): now also M3.3
- net GPIO 27: now reaches U4LEFT.7 (VCC_IO)
- net GPIO 27: now also U1.6 (GPIO27); no longer U1.10 (GPIO32)
- net GPIO 26: now reaches U4LEFT.8 (GND)
- net GPIO 26: now also U1.7 (GPIO26); no longer U1.11 (GPIO35)
- net GPIO 36: now reaches U1.14 (GPIO36)
- net GPIO 21: now reaches U1.26 (GPIO21), U2.5 (SDA)
- net GPIO 22: now reaches U1.29 (GPIO22), U2.4 (SCL)
- net GPIO 12: now reaches U1.4 (GPIO12)
- net GPIO 12: now also U4LEFT.2 (GND)
- net GPIO 14: now reaches U1.5 (GPIO14)
- net GPIO 14: now also U4LEFT.3 (A2)
- net GPIO 25: now reaches U1.8 (GPIO25)
- net GPIO 25: now also U3RIGHT.1 (VM)
- net GPIO 33: now reaches U1.9 (GPIO33)
- net GPIO 33: now also U3RIGHT.2 (GND)
- new net GPIO 15: R1.2, R2.1
- new net GPIO 2: U4LEFT.1 (VM)
- new net GPIO 32: U1.10 (GPIO32), U3RIGHT.3 (A2)
- new net GPIO 34: U1.12 (GPIO34)
- new net GPIO 35: U1.11 (GPIO35)
- new net GPIO 39: U1.13 (GPIO39)
- no-connect marks 0 -> 11
Other:
- note added: "Microcontroller ESP-32"
- note added: "Motor Control Left"
- note added: "Motor Control Right"
- note added: "Power Supply"
- note added: "Tilt Sensor"
- note added: "Voltage divider for battery voltage measurement"
- moved on the sheet: BT1, C1, J2, M2, M3, U1, U2, U3RIGHT, U4LEFT

Commit message: Added circuit changes
Connections:
- net GPIO 15: now also U1.18 (GPIO15)
- net GPIO 16: now also U1.21 (GPIO16)
- net GPIO 17: now also U1.22 (GPIO17)
- net GPIO 2: now also U1.19 (GPIO2)
- net at U3RIGHT.4 (A1): now also M2.1
- net at U3RIGHT.5 (B1): now also M2.4
- net at U3RIGHT.6 (B2): now also M2.3
- net at U4LEFT.4 (A1): now also M3.1
- net at U4LEFT.5 (B1): now also M3.4
- net at U4LEFT.6 (B2): now also M3.3
- net GPIO 34: no longer names the net of U1.12 (GPIO34)
- net GPIO 35: no longer names the net of U1.11 (GPIO35)
- net GPIO 36: no longer names the net of U1.14 (GPIO36)
- net GPIO 39: no longer names the net of U1.13 (GPIO39)
- no-connect marks 11 -> 19
Changed lines of the file:
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@@
+	)
+	(no_connect
+		(at 99.06 116.84)
+	)
+	(no_connect
+		(at 99.06 91.44)
+	)
+	(no_connect
+		(at 99.06 106.68)
 	)
 	(no_connect
@@
 	)
 	(no_connect
+		(at 99.06 88.9)
+	)
+	(no_connect
+		(at 99.06 119.38)
+	)
+	(no_connect
 		(at 158.75 86.36)
 	)
@@
 	)
 	(no_connect
+		(at 99.06 99.06)
+	)
+	(no_connect
+		(at 99.06 109.22)
+	)
+	(no_connect
 		(at 127 124.46)
 	)
@@
 	)
 	(no_connect
+		(at 99.06 111.76)
+	)
+	(no_connect
 		(at 157.48 40.64)
 	)
@@
 	(wire
 		(pts
+			(xy 90.17 104.14) (xy 99.06 104.14)
+		)
+		(stroke
+			(width 0)
+			(type default)
+		)
+	)
+	(wire
+		(pts
 			(xy 191.77 43.18) (xy 175.26 43.18)
 		)
@@
 	(wire
 		(pts
+			(xy 90.17 93.98) (xy 99.06 93.98)
+		)
+		(stroke
+			(width 0)
+			(type default)
+		)
+	)
+	(wire
+		(pts
 			(xy 176.53 76.2) (xy 180.34 76.2)
 		)
@@
 	(wire
 		(pts
-			(xy 127 119.38) (xy 135.89 119.38)
-		)
-		(stroke
-			(width 0)
-			(type default)
-		)
-	)
-	(wire
-		(pts
 			(xy 175.26 48.26) (xy 179.07 48.26)
 		)
@@
 	(wire
 		(pts
+			(xy 90.17 101.6) (xy 99.06 101.6)
+		)
+		(stroke
+			(width 0)
+			(type default)
+		)
+	)
+	(wire
+		(pts
 			(xy 194.31 81.28) (xy 176.53 81.28)
 		)
@@
 	(wire
 		(pts
-			(xy 127 114.3) (xy 135.89 114.3)
-		)
-		(stroke
-			(width 0)
-			(type default)
-		)
-	)
-	(wire
-		(pts
 			(xy 193.04 38.1) (xy 175.26 38.1)
 		)
@@
 	(wire
 		(pts
-			(xy 127 121.92) (xy 135.89 121.92)
-		)
-		(stroke
-			(width 0)
-			(type default)
-		)
-	)
-	(wire
-		(pts
 			(xy 111.76 27.94) (xy 107.95 27.94)
 		)
@@
 	(wire
 		(pts
-			(xy 127 116.84) (xy 135.89 116.84)
-		)
-		(stroke
-			(width 0)
-			(type default)
-		)
-	)
-	(wire
-		(pts
 			(xy 148.59 48.26) (xy 157.48 48.26)
 		)
@@
 		(pts
 			(xy 123.19 27.94) (xy 123.19 40.64)
+		)
+		(stroke
+			(width 0)
+			(type default)
+		)
+	)
+	(wire
+		(pts
+			(xy 90.17 96.52) (xy 99.06 96.52)
 		)
 		(stroke
@@
 		)
 	)
-	(label "GPIO 34"
-		(at 128.27 116.84 0)
-		(effects
-			(font
-				(size 1.27 1.27)
-			)
-			(justify left bottom)
-		)
-	)
 	(label "GPIO 22"
 		(at 68.58 91.44 0)
@@
 		)
 	)
-	(label "GPIO 39"
-		(at 128.27 119.38 0)
+	(label "GPIO 16"
+		(at 90.17 101.6 0)
 		(effects
 			(font
@@
 		)
 	)
+	(label "GPIO 15"
+		(at 90.17 93.98 0)
+		(effects
+			(font
+				(size 1.27 1.27)
+			)
+			(justify left bottom)
+		)
+	)
 	(label "GPIO 16"
 		(at 149.86 91.44 0)
@@
 		)
 	)
+	(label "GPIO 17"
+		(at 90.17 104.14 0)
+		(effects
+			(font
+				(size 1.27 1.27)
+			)
+			(justify left bottom)
+		)
+	)
 	(label "GPIO 21"
 		(at 68.58 88.9 0)
@@
 		)
 	)
-	(label "GPIO 36"
-		(at 128.27 121.92 0)
-		(effects
-			(font
-				(size 1.27 1.27)
-			)
-			(justify left bottom)
-		)
-	)
 	(label "GPIO 22"
 		(at 90.17 121.92 0)
@@
 		)
 	)
-	(label "GPIO 35"
-		(at 128.27 114.3 0)
-		(effects
-			(font
-				(size 1.27 1.27)
-			)
-			(justify left bottom)
-		)
-	)
 	(label "GPIO 26"
 		(at 148.59 50.8 0)
@@
 		(effects
 			(font
+				(size 1.27 1.27)
+			)
+			(justify left bottom)
+		)
+	)
+	(label "GPIO 2"
+		(at 90.17 96.52 0)
+		(effects
+			(font
