File: Schematic/Schaltplan.kicad_sch (KiCad schematic)
At the start: 11 parts, among them J2 Buck Converter, M2 Stepper_Motor_bipolar, M3 Stepper_Motor_bipolar

Commit message: added resistor values to schematic
Parts:
- R1: value R -> 32k
- R2: value R -> 10k
Connections:
- net at U3RIGHT.4 (A1): now also M2.1
- net at U3RIGHT.5 (B1): now also M2.4
- net at U3RIGHT.6 (B2): now also M2.3
- net at U4LEFT.4 (A1): now also M3.1
- net at U4LEFT.5 (B1): now also M3.4
- net at U4LEFT.6 (B2): now also M3.3
- no-connect marks 19 -> 25
Changed lines of the file:
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@@
+	)
+	(no_connect
+		(at 127 114.3)
 	)
 	(no_connect
@@
 	)
 	(no_connect
+		(at 127 93.98)
+	)
+	(no_connect
+		(at 127 119.38)
+	)
+	(no_connect
 		(at 99.06 106.68)
 	)
@@
 	)
 	(no_connect
+		(at 127 116.84)
+	)
+	(no_connect
 		(at 68.58 96.52)
 	)
@@
 	)
 	(no_connect
+		(at 99.06 124.46)
+	)
+	(no_connect
 		(at 68.58 81.28)
 	)
@@
 	(no_connect
 		(at 99.06 111.76)
+	)
+	(no_connect
+		(at 127 121.92)
 	)
 	(no_connect
@@
 			)
 		)
-		(property "Value" "R"
+		(property "Value" "10k"
 			(at 55.88 45.7199 0)
 			(show_name no)
@@
 			)
 		)
-		(property "Value" "R"
+		(property "Value" "32k"
 			(at 55.88 34.2899 0)
 			(show_name no)
